File: eda/IMU.kicad_sch (KiCad schematic)
At the start: 7 parts, among them IC1 ICM-42688-P

Commit message: Add Rev B: routed layout and fab package (Diode 99bcdad)
Imports the completed Rev B board from code.diode.computer/lena/b/string-gauge-daq
at commit 99bcdad.

- Design source: placed, routed and poured 99 x 76 mm 4-layer layout
  (DRC 0 errors / 0 unconnected), AUX fault clamps D10-D13, D6/D7 changed to
  RB168MM-40 (1A_40V_LowIR replaces 1A_20V), ICM-42688-P symbol update.
  pcb build: 256 components.
- fab/rev-b/: JLCPCB Gerber zip, Gerbers/drills, BOM/CPL, schematic/assembly
  PDFs, DRC/ERC reports, STEP, IPC-2581, renders. MANIFEST.txt holds SHA-256
  sums (verified on import).
- spec.md/README.md: Rev B layout and status merged with this repo's own
  edits (test-plan and board-spec references, aux sensor options, run
  metadata).
- .gitignore: anchor docs/ to the repo root so fab/rev-b/docs/ is tracked;
  .gitattributes: store fab/ byte-for-byte.

Not imported: Diode-only import/validation JSONs, the Rev-A KiCad archive zip,
.lfsconfig, and the unused STM32F446RETx symbol.

Co-Authored-By: Claude Opus 5.5 <noreply@anthropic.com>
Connections:
- net GND: now also IC1.9 (INT2_/_FSYNC_/_CLKIN)
- no-connect marks 1 -> 0
Changed lines of the file:
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@@
 	(generator_version "10.0")
 	(paper "A4")
-	(no_connect
-		(at 123.19 90.17)
-	)
 	(wire
 		(pts
@@
 	(wire
 		(pts
+			(xy 123.19 90.17) (xy 128.27 90.17)
+		)
+		(stroke
+			(width 0)
+			(type default)
+		)
+	)
+	(wire
+		(pts
 			(xy 67.31 74.93) (xy 67.31 59.69)
 		)
@@
 		(pts
 			(xy 172.72 90.17) (xy 172.72 92.71)
+		)
+		(stroke
+			(width 0)
+			(type default)
+		)
+	)
+	(wire
+		(pts
+			(xy 128.27 90.17) (xy 128.27 113.03)
 		)
 		(stroke
@@
 					(unit 1)
 				)
+			)
+		)
+	)
+	(symbol
+		(lib_id "GND")
+		(at 128.27 113.03 0)
+		(unit 1)
+		(body_style 1)
+		(exclude_from_sim no)
+		(in_bom yes)
+		(on_board yes)
+		(in_pos_files yes)
+		(dnp no)
+		(fields_autoplaced yes)
+		(property "Reference" "#PWRad620423ccf85d6c9eacfb81d6e66c63"
+			(at 128.27 113.03 0)
+			(hide yes)
+			(show_name no)
+			(do_not_autoplace no)
+			(effects
+				(font
+					(size 1.27 1.27)
+				)
+			)
+		)
+		(property "Value" "GND"
+			(at 128.27 116.84 0)
+			(show_name no)
+			(do_not_autoplace no)
+			(effects
+				(font
+					(size 1.27 1.27)
+				)
+			)
+		)
+		(property "Footprint" ""
+			(at 128.27 113.03 0)
+			(hide yes)
+			(show_name no)
+			(do_not_autoplace no)
+			(effects
+				(font
+					(size 1.27 1.27)
+				)
+			)
+		)
+		(property "Datasheet" ""
+			(at 128.27 113.03 0)
+			(hide yes)
+			(show_name no)
+			(do_not_autoplace no)
+			(effects
+				(font
+					(size 1.27 1.27)
+				)
+			)
+		)
+		(property "Description" "Power symbol creates a global label with name \"GND\" , ground"
+			(at 128.27 113.03 0)
+			(hide yes)
+			(show_name no)
+			(do_not_autoplace no)
+			(effects
+				(font
+					(size 1.27 1.27)
+				)
+			)
+		)
+		(property "ki_keywords" "global power"
+			(at 128.27 113.03 0)
+			(hide yes)
+			(show_name no)
+			(do_not_autoplace no)
+			(effects
+				(font
+					(size 1.27 1.27)
+				)
+			)
+		)
+		(pin "1"
+		)
+		(instances
+			(project "suspension-load-daq"
+				(path "/513d9cc1-d27a-514d-a37c-2f1ca04dddfa/748b5ba0-a895-5c4f-9346-840ef80e97d5"
+					(reference "#PWRad620423ccf85d6c9eacfb81d6e66c63")
+					(unit 1)
+				)
