File: eda/suspension-load-daq.kicad_sch (KiCad schematic)
At the start: 221 parts, among them J1 B3B-PH-K-S, J10 B6B-PH-K-S, J11 B6B-PH-K-S, J12 B6B-PH-K-S, J13 2.54mm 5 x 2 THT Vertical Male, J14 TC2030-NL_CTX, J15 USB4105, J16 B4B-PH-K-S, J17 DM3D-SF, J2 B3B-PH-K-S, J3 B3B-PH-K-S, J4 B3B-PH-K-S, J5 B6B-PH-K-S, J6 B6B-PH-K-S, J7 B6B-PH-K-S, J8 B6B-PH-K-S, J9 B6B-PH-K-S, Q1 PJE138K_R1_00001, Q2 PJE138K_R1_00001, Q3 PJE138K_R1_00001, Q4 PJE138K_R1_00001, Q5 PJE138K_R1_00001, Q6 PJE138K_R1_00001, Q7 PJE138K_R1_00001, Q8 PJE138K_R1_00001, SW1 KMR211NGLFS, U2 LT3042xMSE, U3 STM32F412CEU6, U6 LP5907MFX-3.3, U7 ADS131M08xPBS, Y1 8MHz 10pF

Commit message: Add Rev B: routed layout and fab package (Diode 99bcdad)
Imports the completed Rev B board from code.diode.computer/lena/b/string-gauge-daq
at commit 99bcdad.

- Design source: placed, routed and poured 99 x 76 mm 4-layer layout
  (DRC 0 errors / 0 unconnected), AUX fault clamps D10-D13, D6/D7 changed to
  RB168MM-40 (1A_40V_LowIR replaces 1A_20V), ICM-42688-P symbol update.
  pcb build: 256 components.
- fab/rev-b/: JLCPCB Gerber zip, Gerbers/drills, BOM/CPL, schematic/assembly
  PDFs, DRC/ERC reports, STEP, IPC-2581, renders. MANIFEST.txt holds SHA-256
  sums (verified on import).
- spec.md/README.md: Rev B layout and status merged with this repo's own
  edits (test-plan and board-spec references, aux sensor options, run
  metadata).
- .gitignore: anchor docs/ to the repo root so fab/rev-b/docs/ is tracked;
  .gitattributes: store fab/ byte-for-byte.

Not imported: Diode-only import/validation JSONs, the Rev-A KiCad archive zip,
.lfsconfig, and the unused STM32F446RETx symbol.

Co-Authored-By: Claude Opus 5.5 <noreply@anthropic.com>
Parts:
- added D10, D11, D12, D13: 200mA 30V Schottky Rectifier, stdlib_kicad-footprints_Diode_SMD:D_SOD-323, symbol D_Schottky_Small
- D6: value 1A 20V Schottky Rectifier -> 1A 40V Low-IR Schottky; footprint lena_b_string-gauge-daq_components_1A_20V_Schottky_Rectifier:D_SOD-123F -> lena_b_string-gauge-daq_components_1A_40V_LowIR_Schottky_Rectifier:D_SOD-123F; Path SHEET_8C6BE9B8_106B_5398_B524_BBD11DE1AE5D.D6.1A_20V_Schott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 -> SHEET_8C6BE9B8_106B_5398_B524_BBD11DE1AE5D.D6.1A_40V_LowIR_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
- D7: value 1A 20V Schottky Rectifier -> 1A 40V Low-IR Schottky; footprint lena_b_string-gauge-daq_components_1A_20V_Schottky_Rectifier:D_SOD-123F -> lena_b_string-gauge-daq_components_1A_40V_LowIR_Schottky_Rectifier:D_SOD-123F; Path SHEET_350DCEED_0515_510A_88B9_110E895832F4.D7.1A_20V_Schott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 -> SHEET_350DCEED_0515_510A_88B9_110E895832F4.D7.1A_40V_LowIR_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
Connections:
- net H1.P1 is gone; now on net GND: H1.1
- net H2.P1 is gone; now on net GND: H2.1
- net H3.P1 is gone; now on net GND: H3.1
- net H4.P1 is gone; now on net GND: H4.1
- net AUX1: now also D10.2 (A)
- net AUX2: now also D11.2 (A)
- net AUX3: now also D12.2 (A)
- net AUX4: now also D13.2 (A)
- net V3V3: now also D10.1 (K), D11.1 (K), D12.1 (K), D13.1 (K)
