File: eda/suspension-load-daq.kicad_sch (KiCad schematic)
At the start: 225 parts, among them J1 B3B-PH-K-S, J10 B6B-PH-K-S, J11 B6B-PH-K-S, J12 B6B-PH-K-S, J13 2.54mm 5 x 2 THT Vertical Male, J14 TC2030-NL_CTX, J15 USB4105, J16 B4B-PH-K-S, J17 DM3D-SF, J2 B3B-PH-K-S, J3 B3B-PH-K-S, J4 B3B-PH-K-S, J5 B6B-PH-K-S, J6 B6B-PH-K-S, J7 B6B-PH-K-S, J8 B6B-PH-K-S, J9 B6B-PH-K-S, Q1 PJE138K_R1_00001, Q2 PJE138K_R1_00001, Q3 PJE138K_R1_00001, Q4 PJE138K_R1_00001, Q5 PJE138K_R1_00001, Q6 PJE138K_R1_00001, Q7 PJE138K_R1_00001, Q8 PJE138K_R1_00001, SW1 KMR211NGLFS, U2 LT3042xMSE, U3 STM32F412CEU6, U6 LP5907MFX-3.3, U7 ADS131M08xPBS, Y1 8MHz 10pF

Commit message: did not cook mb
Parts:
- D4: value LED BLUE -> LED YELLOW
- R1, R3, R5, R7: value 18k 1% -> 16.9k 1%
- R86: value 2.2k -> 1k
Connections:
- net V5: no longer JP1.3, JP2.3, JP3.3, JP4.3
- net V5_BUCK: now also JP1.3, JP2.3, JP3.3, JP4.3
