File: eda/suspension-load-daq.kicad_pcb (KiCad board)
At the start: 4 copper layers, 99 x 76 mm, 256 parts, among them IC1 ICM-42688-P, J1 B3B-PH-K-S, J10 B6B-PH-K-S, J11 B6B-PH-K-S, J12 B6B-PH-K-S, J13 2.54mm 5 x 2 THT Vertical Male, J14 TC2030-NL_CTX, J15 USB4105, J16 B4B-PH-K-S, J17 DM3D-SF, J2 B3B-PH-K-S, J3 B3B-PH-K-S, J4 B3B-PH-K-S, J5 B6B-PH-K-S, J6 B6B-PH-K-S, J7 B6B-PH-K-S, J8 B6B-PH-K-S, J9 B6B-PH-K-S, Q1 PJE138K_R1_00001, Q2 PJE138K_R1_00001, Q3 PJE138K_R1_00001, Q4 PJE138K_R1_00001, Q5 PJE138K_R1_00001, Q6 PJE138K_R1_00001, Q7 PJE138K_R1_00001, Q8 PJE138K_R1_00001, SW1 KMR211NGLFS, U1 TCAN1462VDRBRQ1, U2 LT3042xMSE, U3 STM32F412CEU6, U4 TPSM33610S5QRDNRQ1, U5 TPS74501PDRVR, U6 LP5907MFX-3.3, U7 ADS131M08xPBS, Y1 8MHz 10pF

Commit message: update
Other:
- board text added: "+"
- board text added: "1 3V3 2 5V 3 GND 4 GND 5 TX 6 RX 7 SCL 8 SDA"
- board text added: "120R"
- board text added: "3V3"
- board text added: "3V3A"
- board text added: "5V"
- board text added: "9-16 V"
- board text added: "CAL DATE"
- board text added: "CANH"
- board text added: "CANL"
- board text added: "CLKIN"
- board text added: "CORNER"
- board text added: "DRDY"
- board text added: "EXC"
- board text added: "GND"
- board text added: "IN+"
- board text added: "IN-"
- board text added: "JP1-4 AUX SUPPLY 1-2 VDDA / 2-3 5V JP5-12 BRIDGED = HALF BRIDGE JP13 BRIDGED = CAN 120R TERM"
- board text added: "PWR / CAN"
- board text added: "QTR"
- board text added: "S/N"
- board text added: "SIG"
- board text added: "SUSPENSION LOAD DAQ v1.0 OLIN BAJA 2026-10 LA"
- board text added: "SUSPENSION STRAIN LOGGER OLIN BAJA 2026"
- board text added: "V+"
- board text added: "VIN+"
- board text removed: "REV B"
- board text removed: "SUSPENSION STRAIN LOGGER"
